File: hardware/modem_breakout/modem_breakout.kicad_pcb (KiCad board)
At the start: 4 copper layers, 48.3 x 85.1 mm, 73 parts, among them J1 2016504-1, J2 NSIM-7-A, J3 54-00166, J4 Conn_01x01, J5 Conn_01x07, J6 Conn_01x01, Q1 BSS138, Q2 DTC043ZEBTL, U1 EC25AFA-512-STD, U2 TXS0108EPWR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

Commit message: finalize testbench design
Parts:
- added C39: 100nf, Capacitor_SMD:C_0805_2012Metric_Pad1.18x1.45mm_HandSolder, F.Cu at (137.6, 108.7)
- added Q3: DTC043ZEBTL, footprints:SOTFL50P160X85-3N, F.Cu at (141.7, 113.2)
- added R14: 10k, Capacitor_SMD:C_0805_2012Metric_Pad1.18x1.45mm_HandSolder, F.Cu at (144.6, 108.8)
- added R15: 10k, Capacitor_SMD:C_0805_2012Metric_Pad1.18x1.45mm_HandSolder, F.Cu at (172.8, 68.3)
- J4, J6: value Conn_01x01 -> Conn_01x02; footprint Connector_PinHeader_2.54mm:PinHeader_1x01_P2.54mm_Vertical -> Connector_PinHeader_2.54mm:PinHeader_1x02_P2.54mm_Vertical
- moved J4 22.9 mm to (153.9, 124.9), turned to -90 degrees
- moved J6 11.9 mm to (174.2, 61.4)
Connections:
- U1 pad 21: unconnected-(U1-PWRKEY-Pad21) -> Net-(U1-PWRKEY)
Routing:
- net CODEC_RESET: track 11.1 -> 47.2 mm
- net STATUS: track 0.00 -> 31.5 mm
- net EC_PWRKEY: track 0.00 -> 19.1 mm
- net Net-(U1-PWRKEY): track 0.00 -> 15.8 mm
- net +3.3V: track 17.9 -> 21.2 mm, vias 22 -> 24
- net GND: track 125.8 -> 127.6 mm, vias 250 -> 252
- net EC_PWR_EN: track 8.42 -> 8.98 mm
Other:
- board text added: "CODEC_RESET"
- board text added: "CTS"
- board text added: "DCD"
- board text added: "DTR"
- board text added: "PWRKEY"
- board text added: "PWR_EN"
- board text added: "RING"
- board text added: "RTS"
- board text added: "RX"
- board text added: "STATUS"
- board text added: "TX"

Commit message: final - ordered
Parts:
- removed J5: Conn_01x07, Connector_PinHeader_2.54mm:PinHeader_1x07_P2.54mm_Vertical
- added GND: Conn_01x08, Connector_PinHeader_2.54mm:PinHeader_1x08_P2.54mm_Vertical, F.Cu at (130.8, 50.6)
